File: board/board.kicad_pcb (KiCad board)
At the start: 2 copper layers, 21 x 13 mm, 1 part

Commit message: initial
Parts:
- added C1: 100nF, Capacitor_SMD:C_0402_1005Metric, F.Cu at (161.7, 101.7)
- added C2: 10uF, Capacitor_SMD:C_0402_1005Metric, F.Cu at (160.7, 101.7)
- added C3: 100nF, Capacitor_SMD:C_0402_1005Metric, F.Cu at (161.7, 99.8)
- added C4: 100nF, Capacitor_SMD:C_0402_1005Metric, F.Cu at (161.7, 94.0)
- added C5: 10uF, Capacitor_SMD:C_0402_1005Metric, F.Cu at (161.7, 92.2)
- added C6: 100nF, Capacitor_SMD:C_0402_1005Metric, F.Cu at (160.7, 92.2)
- added C7: 8pF, Capacitor_SMD:C_0402_1005Metric, F.Cu at (177.6, 101.2)
- added C8: 8pF, Capacitor_SMD:C_0402_1005Metric, F.Cu at (179.0, 101.2)
- added J1: 008_USB, on_edge:on_edge_2x05_host, F.Cu at (185.0, 96.5)
- added J2: 008_USB, on_edge:on_edge_2x05_device, F.Cu at (140.0, 96.5)
- added J3: B0505M-2WR2, Connector_PinHeader_2.54mm:PinHeader_1x04_P2.54mm_Vertical, F.Cu at (148.8, 97.6)
- added U1: ADUM3166, Package_SO:SOIC-20W_7.5x12.8mm_P1.27mm, F.Cu at (168.8, 96.7)
- added Y1: Crystal_GND24_Small, Crystal:Crystal_SMD_3225-4Pin_3.2x2.5mm, F.Cu at (177.6, 98.5)
- LOGO1: moved to B.Cu
- moved LOGO1 19.0 mm to (168.8, 96.7), turned to 180 degrees
Routing:
- net /dcdc/GND2: track 0.00 -> 55.3 mm, vias 0 -> 25
- net /dcdc/GND1: track 0.00 -> 48.1 mm, vias 0 -> 25
- net /dcdc/5Vout: track 0.00 -> 34.1 mm, vias 0 -> 1
- net /iso/D-: track 0.00 -> 33.7 mm, vias 0 -> 2
- net /iso/D+: track 0.00 -> 33.5 mm, vias 0 -> 2
- net /dcdc/5Vin: track 0.00 -> 29.1 mm, vias 0 -> 1
- net Net-(U1-XO2): track 0.00 -> 15.9 mm
- net Net-(U1-XI2): track 0.00 -> 13.8 mm
- net /iso/DD-: track 0.00 -> 13.6 mm
- net /iso/DD+: track 0.00 -> 11.9 mm
- net /iso/VDD1: track 0.00 -> 5.65 mm
- net /iso/VDD2: track 0.00 -> 5.60 mm
- added copper zone on B.Cu, net /dcdc/GND1
- added copper zone on F.Cu, net /dcdc/GND1
- added copper zone on B.Cu, net /dcdc/GND2
- added copper zone on F.Cu, net /dcdc/GND2
Other:
- board size 21 x 13 mm -> 45 x 13 mm
- board text added: "osf.008"
- board text added: "osf.b156.v1.0"
