File: board/iso.kicad_sch (KiCad schematic)
At the start: 10 parts, among them U1 ADUM3166, Y1 Crystal_GND24_Small

Commit message: fixed chip package
Parts:
- U1: footprint Package_SO:SOIC-20W_7.5x12.8mm_P1.27mm -> Package_SO:SSOP-20_5.3x7.2mm_P0.65mm
Changed lines of the file:
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@@
       (effects (font (size 1.27 1.27)))
     )
-    (property "Footprint" "Package_SO:SOIC-20W_7.5x12.8mm_P1.27mm" (at 135.89 85.09 0)
+    (property "Footprint" "Package_SO:SSOP-20_5.3x7.2mm_P0.65mm" (at 135.89 85.09 0)
       (effects (font (size 1.27 1.27)) hide)
     )
